File: m78.kicad_pcb (KiCad board)
At the start: 2 copper layers, 243.2 x 143 mm, 161 parts, among them SW1 mx, SW10 mx, SW11 mx, SW12 mx, SW13 mx, SW14 mx, SW15 mx, SW16 mx, SW17 mx, SW18 mx, SW19 mx, SW2 mx, SW20 mx, SW21 mx, SW22 mx, SW23 mx, SW24 mx, SW25 mx, SW26 mx, SW27 mx, SW28 mx, SW29 mx, SW3 mx, SW30 mx, SW31 mx, SW32 mx, SW33 mx, SW34 mx, SW35 mx, SW36 mx, SW37 mx, SW38 mx, SW39 mx, SW4 mx, SW40 mx, SW41 mx, SW42 mx, SW43 mx, SW44 mx, SW45 mx, SW46 mx, SW47 mx, SW48 mx, SW49 mx, SW5 mx, SW50 mx, SW51 mx, SW52 mx, SW53 mx, SW54 mx, SW55 mx, SW56 mx, SW57 mx, SW58 mx, SW59 mx, SW6 mx, SW60 mx, SW61 mx, SW62 mx, SW63 mx, SW64 mx, SW65 mx, SW66 mx, SW67 mx, SW68 mx, SW69 mx, SW7 mx, SW70 mx, SW71 mx, SW72 mx, SW73 mx, SW74 mx, SW75 mx, SW76 mx, SW77 mx, SW78 mx, SW8 mx, SW9 mx, U1 Teensy2.0

Commit message: rename to something more sensible
Parts:
- added D81: LED, LED_THT:LED_D3.0mm_Clear, F.Cu at (213.8, 30.8)
- added R3: R, Resistor_THT:R_Axial_DIN0207_L6.3mm_D2.5mm_P7.62mm_Horizontal, F.Cu at (219.7, 31.1)
- D1, D10, D11, D13, D14, D15, D16, D17, D19, D2, D20, D21, D22, D23, D25, D26, D27, D28, D29, D3, D31, D32, D33, D34, D35, D37, D38, D39, D4, D40, D41, D43, D44, D45, D46, D47, D49, D5, D50, D51, D52, D53, D55, D56, D57, D58, D59, D61, D62, D63, D64, D65, D68, D69, D7, D70, D71, D73, D74, D75, D76, D77, D8, D9: footprint test-k:diode_v -> m78:diode_v
- D12, D18, D24, D30, D36, D42, D48, D54, D6, D60, D66, D72, D78: footprint Diode_THT:D_DO-35_SOD27_P7.62mm_Horizontal -> m78:diode_h
- D67: footprint test-k:diode_v -> m78:diode_h
- U1: value Teensy2.0 -> TEENSY2.0; footprint test-k:Teensy2.0 -> m78:Teensy2.0
- moved U1 33.0 mm to (235.4, 35.9)
- moved D79 0.46 mm to (213.8, 19.1)
- moved D80 0.46 mm to (213.8, 25.4)
Connections:
- U1 pad 14: (no net) -> pwr

Commit message: update
Parts:
- D12, D18, D24, D30, D36, D42, D48, D54, D6, D60, D66, D67, D72: footprint m78:diode_h -> m78:diode_v
- SW1, SW10, SW11, SW12, SW13, SW14, SW15, SW16, SW17, SW18, SW19, SW2, SW20, SW21, SW22, SW23, SW24, SW25, SW26, SW27, SW28, SW29, SW3, SW30, SW31, SW32, SW33, SW34, SW35, SW36, SW37, SW38, SW39, SW4, SW40, SW41, SW42, SW43, SW44, SW45, SW46, SW47, SW48, SW49, SW5, SW50, SW51, SW52, SW53, SW54, SW55, SW56, SW57, SW58, SW59, SW6, SW60, SW61, SW62, SW63, SW64, SW65, SW66, SW67, SW68, SW69, SW7, SW70, SW71, SW72, SW73, SW74, SW75, SW76, SW77, SW78, SW8, SW9: footprint Button_Switch_Keyboard:SW_Cherry_MX_1.00u_PCB -> Button_Switch_Keyboard:SW_Cherry_MX_1.00u_Plate
- U1: footprint m78:Teensy2.0 -> m78:Teensy2.0-pins
- moved D78 143.9 mm to (248.1, 154.0), turned to 90 degrees
- moved D72 142.4 mm to (229.1, 154.0), turned to 90 degrees
- moved D66 141.0 mm to (210.0, 154.0), turned to 90 degrees
- moved D60 139.8 mm to (191.0, 154.0), turned to 90 degrees
- moved D54 138.7 mm to (171.9, 154.0), turned to 90 degrees
- moved D77 115.8 mm to (248.1, 134.9), turned to 90 degrees
- moved D71 114.5 mm to (229.1, 134.9), turned to 90 degrees
- moved D65 113.3 mm to (210.0, 134.9), turned to 90 degrees
- moved D59 112.2 mm to (191.0, 134.9), turned to 90 degrees
- moved D53 111.3 mm to (171.9, 134.9), turned to 90 degrees
- moved D76 99.2 mm to (248.1, 115.9), turned to 90 degrees
- moved D70 97.5 mm to (229.1, 115.9), turned to 90 degrees
- moved D64 95.9 mm to (210.0, 115.9), turned to 90 degrees
- moved D58 94.5 mm to (191.0, 115.9), turned to 90 degrees
- moved D75 83.7 mm to (248.1, 96.8), turned to 90 degrees
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Connections:
- U1 pad 10: c1 -> (no net)
- U1 pad 11: c0 -> (no net)
- U1 pad 12: cpp -> c8
- U1 pad 13: f90 -> (no net)
- U1 pad 17: (no net) -> f90
- U1 pad 18: c8 -> cpp
- U1 pad 2: (no net) -> c7
- U1 pad 22: c12 -> r5
- U1 pad 23: r5 -> r4
- U1 pad 24: r4 -> c12
- U1 pad 26: r2 -> r1
- U1 pad 27: r1 -> r0
- U1 pad 28: r0 -> r2
- U1 pad 3: (no net) -> c6
- U1 pad 4: c7 -> c5
- U1 pad 5: c6 -> c4
- U1 pad 6: c5 -> c3
- U1 pad 7: c4 -> c2
- U1 pad 8: c3 -> c0
- U1 pad 9: c2 -> c1
Routing:
- net r5: track 0.00 -> 342.5 mm
- net r4: track 0.00 -> 323.3 mm
- net r3: track 0.00 -> 305.5 mm
- net r2: track 0.00 -> 284.5 mm
- net r1: track 0.00 -> 266.3 mm
- net r0: track 0.00 -> 246.2 mm
- net c0: track 0.00 -> 219.5 mm
- net c1: track 0.00 -> 196.9 mm
- net c8: track 0.00 -> 183.7 mm
- net c2: track 0.00 -> 182.4 mm
- net c9: track 0.00 -> 170.5 mm
- net c3: track 0.00 -> 165.2 mm
- net c10: track 0.00 -> 158.3 mm
- net c11: track 0.00 -> 152.1 mm
- net c4: track 0.00 -> 149.4 mm
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Other:
- board size 243.2 x 143 mm -> 244 x 144 mm
- board text added: "L'essentiel est invisible pour les yeux."

Commit message: diodes in rows
Parts:
- D78: footprint m78:diode_h -> m78:diode_v
- moved D68 186.8 mm to (51.3, 20.6), turned to 270 degrees
- moved D62 165.9 mm to (48.7, 20.6)
- moved D56 161.5 mm to (46.2, 20.6)
- moved D50 150.3 mm to (43.6, 20.6)
- moved D69 149.5 mm to (100.5, 20.6), turned to 270 degrees
- moved D63 135.8 mm to (97.6, 20.6), turned to 270 degrees
- moved D70 133.8 mm to (136.3, 19.4), turned to 270 degrees
- moved D6 133.5 mm to (36.0, 150.2), turned to 90 degrees
- moved D44 132.2 mm to (41.1, 20.6)
- moved D42 131.8 mm to (150.3, 150.2), turned to 90 degrees
- moved D12 131.0 mm to (55.1, 150.2), turned to 90 degrees
- moved D18 128.6 mm to (74.1, 150.2), turned to 90 degrees
- moved D36 127.8 mm to (131.3, 150.2), turned to 90 degrees
- moved D24 127.5 mm to (93.2, 150.2), turned to 90 degrees
- moved D71 126.8 mm to (177.0, 19.4), turned to 270 degrees
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Connections:
- D1 pad 1: c0 -> r0
- D10 pad 1: c1 -> r3
- D11 pad 1: c1 -> r4
- D12 pad 1: c1 -> r5
- D13 pad 1: c2 -> r0
- D14 pad 1: c2 -> r1
- D15 pad 1: c2 -> r2
- D16 pad 1: c2 -> r3
- D17 pad 1: c2 -> r4
- D18 pad 1: c2 -> r5
- D19 pad 1: c3 -> r0
- D2 pad 1: c0 -> r1
- D20 pad 1: c3 -> r1
- D21 pad 1: c3 -> r2
- D22 pad 1: c3 -> r3
- D23 pad 1: c3 -> r4
- D24 pad 1: c3 -> r5
- D25 pad 1: c4 -> r0
- D26 pad 1: c4 -> r1
- D27 pad 1: c4 -> r2
- D28 pad 1: c4 -> r3
- D29 pad 1: c4 -> r4
- D3 pad 1: c0 -> r2
- D30 pad 1: c4 -> r5
- D31 pad 1: c5 -> r0
- D32 pad 1: c5 -> r1
- D33 pad 1: c5 -> r2
- D34 pad 1: c5 -> r3
- D35 pad 1: c5 -> r4
- D36 pad 1: c5 -> r5
- D37 pad 1: c6 -> r0
- D38 pad 1: c6 -> r1
- D39 pad 1: c6 -> r2
- D4 pad 1: c0 -> r3
- D40 pad 1: c6 -> r3
- D41 pad 1: c6 -> r4
- D42 pad 1: c6 -> r5
- D43 pad 1: c7 -> r0
- D44 pad 1: c7 -> r1
- D45 pad 1: c7 -> r2
- D46 pad 1: c7 -> r3
- D47 pad 1: c7 -> r4
- D48 pad 1: c7 -> r5
- D49 pad 1: c8 -> r0
- D5 pad 1: c0 -> r4
- D50 pad 1: c8 -> r1
- D51 pad 1: c8 -> r2
- D52 pad 1: c8 -> r3
- D53 pad 1: c8 -> r4
- D54 pad 1: c8 -> r5
- D55 pad 1: c9 -> r0
- D56 pad 1: c9 -> r1
- D57 pad 1: c9 -> r2
- D58 pad 1: c9 -> r3
- D59 pad 1: c9 -> r4
- D6 pad 1: c0 -> r5
- D60 pad 1: c9 -> r5
- D61 pad 1: c10 -> r0
- D62 pad 1: c10 -> r1
- D63 pad 1: c10 -> r2
- D64 pad 1: c10 -> r3
- D65 pad 1: c10 -> r4
- D66 pad 1: c10 -> r5
- D67 pad 1: c11 -> r0
- D68 pad 1: c11 -> r1
- D69 pad 1: c11 -> r2
- D7 pad 1: c1 -> r0
- D70 pad 1: c11 -> r3
- D71 pad 1: c11 -> r4
- D72 pad 1: c11 -> r5
- D73 pad 1: c12 -> r0
- D74 pad 1: c12 -> r1
- D75 pad 1: c12 -> r2
- D76 pad 1: c12 -> r3
- D77 pad 1: c12 -> r4
- D78 pad 1: c12 -> r5
- D8 pad 1: c1 -> r1
- D9 pad 1: c1 -> r2
- SW1 pad 1: r0 -> Net-(D1-Pad2)
- SW1 pad 2: Net-(D1-Pad2) -> c0
- SW10 pad 1: r3 -> Net-(D10-Pad2)
- SW10 pad 2: Net-(D10-Pad2) -> c1
- SW11 pad 1: r4 -> Net-(D11-Pad2)
- SW11 pad 2: Net-(D11-Pad2) -> c1
- SW12 pad 1: r5 -> Net-(D12-Pad2)
- SW12 pad 2: Net-(D12-Pad2) -> c1
- SW13 pad 1: r0 -> Net-(D13-Pad2)
- SW13 pad 2: Net-(D13-Pad2) -> c2
- SW14 pad 1: r1 -> Net-(D14-Pad2)
- SW14 pad 2: Net-(D14-Pad2) -> c2
- SW15 pad 1: r2 -> Net-(D15-Pad2)
- SW15 pad 2: Net-(D15-Pad2) -> c2
- SW16 pad 1: r3 -> Net-(D16-Pad2)
- SW16 pad 2: Net-(D16-Pad2) -> c2
- SW17 pad 1: r4 -> Net-(D17-Pad2)
- SW17 pad 2: Net-(D17-Pad2) -> c2
- SW18 pad 1: r5 -> Net-(D18-Pad2)
- SW18 pad 2: Net-(D18-Pad2) -> c2
- SW19 pad 1: r0 -> Net-(D19-Pad2)
- SW19 pad 2: Net-(D19-Pad2) -> c3
- SW2 pad 1: r1 -> Net-(D2-Pad2)
- SW2 pad 2: Net-(D2-Pad2) -> c0
- SW20 pad 1: r1 -> Net-(D20-Pad2)
- SW20 pad 2: Net-(D20-Pad2) -> c3
- SW21 pad 1: r2 -> Net-(D21-Pad2)
- SW21 pad 2: Net-(D21-Pad2) -> c3
- SW22 pad 1: r3 -> Net-(D22-Pad2)
- SW22 pad 2: Net-(D22-Pad2) -> c3
- SW23 pad 1: r4 -> Net-(D23-Pad2)
- SW23 pad 2: Net-(D23-Pad2) -> c3
- SW24 pad 1: r5 -> Net-(D24-Pad2)
- SW24 pad 2: Net-(D24-Pad2) -> c3
- SW25 pad 1: r0 -> Net-(D25-Pad2)
- SW25 pad 2: Net-(D25-Pad2) -> c4
- SW26 pad 1: r1 -> Net-(D26-Pad2)
- SW26 pad 2: Net-(D26-Pad2) -> c4
- SW27 pad 1: r2 -> Net-(D27-Pad2)
- SW27 pad 2: Net-(D27-Pad2) -> c4
- SW28 pad 1: r3 -> Net-(D28-Pad2)
- SW28 pad 2: Net-(D28-Pad2) -> c4
- SW29 pad 1: r4 -> Net-(D29-Pad2)
- SW29 pad 2: Net-(D29-Pad2) -> c4
- SW3 pad 1: r2 -> Net-(D3-Pad2)
- SW3 pad 2: Net-(D3-Pad2) -> c0
- SW30 pad 1: r5 -> Net-(D30-Pad2)
- SW30 pad 2: Net-(D30-Pad2) -> c4
- SW31 pad 1: r0 -> Net-(D31-Pad2)
- SW31 pad 2: Net-(D31-Pad2) -> c5
- SW32 pad 1: r1 -> Net-(D32-Pad2)
- SW32 pad 2: Net-(D32-Pad2) -> c5
- SW33 pad 1: r2 -> Net-(D33-Pad2)
- SW33 pad 2: Net-(D33-Pad2) -> c5
- SW34 pad 1: r3 -> Net-(D34-Pad2)
- SW34 pad 2: Net-(D34-Pad2) -> c5
- SW35 pad 1: r4 -> Net-(D35-Pad2)
- SW35 pad 2: Net-(D35-Pad2) -> c5
- SW36 pad 1: r5 -> Net-(D36-Pad2)
- SW36 pad 2: Net-(D36-Pad2) -> c5
- SW37 pad 1: r0 -> Net-(D37-Pad2)
- SW37 pad 2: Net-(D37-Pad2) -> c6
- SW38 pad 1: r1 -> Net-(D38-Pad2)
- SW38 pad 2: Net-(D38-Pad2) -> c6
- SW39 pad 1: r2 -> Net-(D39-Pad2)
- SW39 pad 2: Net-(D39-Pad2) -> c6
- SW4 pad 1: r3 -> Net-(D4-Pad2)
- SW4 pad 2: Net-(D4-Pad2) -> c0
- SW40 pad 1: r3 -> Net-(D40-Pad2)
- SW40 pad 2: Net-(D40-Pad2) -> c6
- SW41 pad 1: r4 -> Net-(D41-Pad2)
- SW41 pad 2: Net-(D41-Pad2) -> c6
- SW42 pad 1: r5 -> Net-(D42-Pad2)
- SW42 pad 2: Net-(D42-Pad2) -> c6
- SW43 pad 1: r0 -> Net-(D43-Pad2)
- SW43 pad 2: Net-(D43-Pad2) -> c7
- SW44 pad 1: r1 -> Net-(D44-Pad2)
- SW44 pad 2: Net-(D44-Pad2) -> c7
- SW45 pad 1: r2 -> Net-(D45-Pad2)
- SW45 pad 2: Net-(D45-Pad2) -> c7
- SW46 pad 1: r3 -> Net-(D46-Pad2)
- SW46 pad 2: Net-(D46-Pad2) -> c7
- SW47 pad 1: r4 -> Net-(D47-Pad2)
- SW47 pad 2: Net-(D47-Pad2) -> c7
- SW48 pad 1: r5 -> Net-(D48-Pad2)
- SW48 pad 2: Net-(D48-Pad2) -> c7
- SW49 pad 1: r0 -> Net-(D49-Pad2)
- SW49 pad 2: Net-(D49-Pad2) -> c8
- SW5 pad 1: r4 -> Net-(D5-Pad2)
- SW5 pad 2: Net-(D5-Pad2) -> c0
- SW50 pad 1: r1 -> Net-(D50-Pad2)
- SW50 pad 2: Net-(D50-Pad2) -> c8
- SW51 pad 1: r2 -> Net-(D51-Pad2)
- SW51 pad 2: Net-(D51-Pad2) -> c8
- SW52 pad 1: r3 -> Net-(D52-Pad2)
- SW52 pad 2: Net-(D52-Pad2) -> c8
- SW53 pad 1: r4 -> Net-(D53-Pad2)
- SW53 pad 2: Net-(D53-Pad2) -> c8
- SW54 pad 1: r5 -> Net-(D54-Pad2)
- SW54 pad 2: Net-(D54-Pad2) -> c8
- SW55 pad 1: r0 -> Net-(D55-Pad2)
- SW55 pad 2: Net-(D55-Pad2) -> c9
- SW56 pad 1: r1 -> Net-(D56-Pad2)
- SW56 pad 2: Net-(D56-Pad2) -> c9
- SW57 pad 1: r2 -> Net-(D57-Pad2)
- SW57 pad 2: Net-(D57-Pad2) -> c9
- SW58 pad 1: r3 -> Net-(D58-Pad2)
- SW58 pad 2: Net-(D58-Pad2) -> c9
- SW59 pad 1: r4 -> Net-(D59-Pad2)
- SW59 pad 2: Net-(D59-Pad2) -> c9
- SW6 pad 1: r5 -> Net-(D6-Pad2)
- SW6 pad 2: Net-(D6-Pad2) -> c0
- SW60 pad 1: r5 -> Net-(D60-Pad2)
- SW60 pad 2: Net-(D60-Pad2) -> c9
- SW61 pad 1: r0 -> Net-(D61-Pad2)
- SW61 pad 2: Net-(D61-Pad2) -> c10
- SW62 pad 1: r1 -> Net-(D62-Pad2)
- SW62 pad 2: Net-(D62-Pad2) -> c10
- SW63 pad 1: r2 -> Net-(D63-Pad2)
- SW63 pad 2: Net-(D63-Pad2) -> c10
- SW64 pad 1: r3 -> Net-(D64-Pad2)
- SW64 pad 2: Net-(D64-Pad2) -> c10
- SW65 pad 1: r4 -> Net-(D65-Pad2)
- SW65 pad 2: Net-(D65-Pad2) -> c10
- SW66 pad 1: r5 -> Net-(D66-Pad2)
- SW66 pad 2: Net-(D66-Pad2) -> c10
- SW67 pad 1: r0 -> Net-(D67-Pad2)
- SW67 pad 2: Net-(D67-Pad2) -> c11
- SW68 pad 1: r1 -> Net-(D68-Pad2)
- SW68 pad 2: Net-(D68-Pad2) -> c11
- SW69 pad 1: r2 -> Net-(D69-Pad2)
- SW69 pad 2: Net-(D69-Pad2) -> c11
- SW7 pad 1: r0 -> Net-(D7-Pad2)
- SW7 pad 2: Net-(D7-Pad2) -> c1
- SW70 pad 1: r3 -> Net-(D70-Pad2)
- SW70 pad 2: Net-(D70-Pad2) -> c11
- SW71 pad 1: r4 -> Net-(D71-Pad2)
- SW71 pad 2: Net-(D71-Pad2) -> c11
- SW72 pad 1: r5 -> Net-(D72-Pad2)
- SW72 pad 2: Net-(D72-Pad2) -> c11
- SW73 pad 1: r0 -> Net-(D73-Pad2)
- SW73 pad 2: Net-(D73-Pad2) -> c12
- SW74 pad 1: r1 -> Net-(D74-Pad2)
- SW74 pad 2: Net-(D74-Pad2) -> c12
- SW75 pad 1: r2 -> Net-(D75-Pad2)
- SW75 pad 2: Net-(D75-Pad2) -> c12
- SW76 pad 1: r3 -> Net-(D76-Pad2)
- SW76 pad 2: Net-(D76-Pad2) -> c12
- SW77 pad 1: r4 -> Net-(D77-Pad2)
- SW77 pad 2: Net-(D77-Pad2) -> c12
- SW78 pad 1: r5 -> Net-(D78-Pad2)
- SW78 pad 2: Net-(D78-Pad2) -> c12
- SW8 pad 1: r1 -> Net-(D8-Pad2)
- SW8 pad 2: Net-(D8-Pad2) -> c1
- SW9 pad 1: r2 -> Net-(D9-Pad2)
- SW9 pad 2: Net-(D9-Pad2) -> c1
Routing:
- net Net-(D68-Pad2): track 4.74 -> 209.8 mm, vias 0 -> 1
- net Net-(D69-Pad2): track 4.74 -> 171.3 mm, vias 0 -> 1
- net Net-(D62-Pad2): track 37.7 -> 192.6 mm, vias 0 -> 1
- net Net-(D63-Pad2): track 4.74 -> 153.7 mm, vias 0 -> 1
- net Net-(D70-Pad2): track 4.74 -> 142.1 mm, vias 0 -> 1
- net Net-(D56-Pad2): track 41.5 -> 175.6 mm, vias 0 -> 1
- net Net-(D64-Pad2): track 4.74 -> 131.3 mm, vias 0 -> 1
- net Net-(D42-Pad2): track 130.6 -> 5.08 mm
- net Net-(D6-Pad2): track 129.1 -> 5.08 mm
- net Net-(D12-Pad2): track 127.2 -> 5.08 mm
- net Net-(D36-Pad2): track 126.1 -> 5.08 mm
- net Net-(D18-Pad2): track 125.3 -> 5.08 mm
- net c6: track 109.4 -> 229.4 mm
- net Net-(D48-Pad2): track 124.9 -> 5.08 mm
- net Net-(D24-Pad2): track 124.8 -> 5.08 mm
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
Commit message: Revert "diodes in rows"
This reverts commit 9845cd0533da21a297a661dd2d085098a01597ee.
Parts:
- D78: footprint m78:diode_v -> m78:diode_h
- moved D68 186.8 mm to (229.1, 77.8), turned to 90 degrees
- moved D62 165.9 mm to (214.5, 25.7)
- moved D56 161.5 mm to (207.6, 25.7)
- moved D50 150.3 mm to (193.8, 25.7)
- moved D69 149.5 mm to (229.1, 96.8), turned to 90 degrees
- moved D63 135.8 mm to (210.0, 96.8), turned to 90 degrees
- moved D70 133.8 mm to (229.1, 115.9), turned to 90 degrees
- moved D6 133.5 mm to (42.1, 16.8), turned to 270 degrees
- moved D44 132.2 mm to (173.2, 25.7)
- moved D42 131.8 mm to (166.3, 19.4), turned to 270 degrees
- moved D12 131.0 mm to (62.8, 19.4), turned to 270 degrees
- moved D18 128.6 mm to (83.5, 21.9), turned to 270 degrees
- moved D36 127.8 mm to (145.6, 23.2), turned to 270 degrees
- moved D24 127.5 mm to (104.2, 23.2), turned to 270 degrees
- moved D71 126.8 mm to (229.1, 134.9), turned to 90 degrees
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Connections:
- D1 pad 1: r0 -> c0
- D10 pad 1: r3 -> c1
- D11 pad 1: r4 -> c1
- D12 pad 1: r5 -> c1
- D13 pad 1: r0 -> c2
- D14 pad 1: r1 -> c2
- D15 pad 1: r2 -> c2
- D16 pad 1: r3 -> c2
- D17 pad 1: r4 -> c2
- D18 pad 1: r5 -> c2
- D19 pad 1: r0 -> c3
- D2 pad 1: r1 -> c0
- D20 pad 1: r1 -> c3
- D21 pad 1: r2 -> c3
- D22 pad 1: r3 -> c3
- D23 pad 1: r4 -> c3
- D24 pad 1: r5 -> c3
- D25 pad 1: r0 -> c4
- D26 pad 1: r1 -> c4
- D27 pad 1: r2 -> c4
- D28 pad 1: r3 -> c4
- D29 pad 1: r4 -> c4
- D3 pad 1: r2 -> c0
- D30 pad 1: r5 -> c4
- D31 pad 1: r0 -> c5
- D32 pad 1: r1 -> c5
- D33 pad 1: r2 -> c5
- D34 pad 1: r3 -> c5
- D35 pad 1: r4 -> c5
- D36 pad 1: r5 -> c5
- D37 pad 1: r0 -> c6
- D38 pad 1: r1 -> c6
- D39 pad 1: r2 -> c6
- D4 pad 1: r3 -> c0
- D40 pad 1: r3 -> c6
- D41 pad 1: r4 -> c6
- D42 pad 1: r5 -> c6
- D43 pad 1: r0 -> c7
- D44 pad 1: r1 -> c7
- D45 pad 1: r2 -> c7
- D46 pad 1: r3 -> c7
- D47 pad 1: r4 -> c7
- D48 pad 1: r5 -> c7
- D49 pad 1: r0 -> c8
- D5 pad 1: r4 -> c0
- D50 pad 1: r1 -> c8
- D51 pad 1: r2 -> c8
- D52 pad 1: r3 -> c8
- D53 pad 1: r4 -> c8
- D54 pad 1: r5 -> c8
- D55 pad 1: r0 -> c9
- D56 pad 1: r1 -> c9
- D57 pad 1: r2 -> c9
- D58 pad 1: r3 -> c9
- D59 pad 1: r4 -> c9
- D6 pad 1: r5 -> c0
- D60 pad 1: r5 -> c9
- D61 pad 1: r0 -> c10
- D62 pad 1: r1 -> c10
- D63 pad 1: r2 -> c10
- D64 pad 1: r3 -> c10
- D65 pad 1: r4 -> c10
- D66 pad 1: r5 -> c10
- D67 pad 1: r0 -> c11
- D68 pad 1: r1 -> c11
- D69 pad 1: r2 -> c11
- D7 pad 1: r0 -> c1
- D70 pad 1: r3 -> c11
- D71 pad 1: r4 -> c11
- D72 pad 1: r5 -> c11
- D73 pad 1: r0 -> c12
- D74 pad 1: r1 -> c12
- D75 pad 1: r2 -> c12
- D76 pad 1: r3 -> c12
- D77 pad 1: r4 -> c12
- D78 pad 1: r5 -> c12
- D8 pad 1: r1 -> c1
- D9 pad 1: r2 -> c1
- SW1 pad 1: Net-(D1-Pad2) -> r0
- SW1 pad 2: c0 -> Net-(D1-Pad2)
- SW10 pad 1: Net-(D10-Pad2) -> r3
- SW10 pad 2: c1 -> Net-(D10-Pad2)
- SW11 pad 1: Net-(D11-Pad2) -> r4
- SW11 pad 2: c1 -> Net-(D11-Pad2)
- SW12 pad 1: Net-(D12-Pad2) -> r5
- SW12 pad 2: c1 -> Net-(D12-Pad2)
- SW13 pad 1: Net-(D13-Pad2) -> r0
- SW13 pad 2: c2 -> Net-(D13-Pad2)
- SW14 pad 1: Net-(D14-Pad2) -> r1
- SW14 pad 2: c2 -> Net-(D14-Pad2)
- SW15 pad 1: Net-(D15-Pad2) -> r2
- SW15 pad 2: c2 -> Net-(D15-Pad2)
- SW16 pad 1: Net-(D16-Pad2) -> r3
- SW16 pad 2: c2 -> Net-(D16-Pad2)
- SW17 pad 1: Net-(D17-Pad2) -> r4
- SW17 pad 2: c2 -> Net-(D17-Pad2)
- SW18 pad 1: Net-(D18-Pad2) -> r5
- SW18 pad 2: c2 -> Net-(D18-Pad2)
- SW19 pad 1: Net-(D19-Pad2) -> r0
- SW19 pad 2: c3 -> Net-(D19-Pad2)
- SW2 pad 1: Net-(D2-Pad2) -> r1
- SW2 pad 2: c0 -> Net-(D2-Pad2)
- SW20 pad 1: Net-(D20-Pad2) -> r1
- SW20 pad 2: c3 -> Net-(D20-Pad2)
- SW21 pad 1: Net-(D21-Pad2) -> r2
- SW21 pad 2: c3 -> Net-(D21-Pad2)
- SW22 pad 1: Net-(D22-Pad2) -> r3
- SW22 pad 2: c3 -> Net-(D22-Pad2)
- SW23 pad 1: Net-(D23-Pad2) -> r4
- SW23 pad 2: c3 -> Net-(D23-Pad2)
- SW24 pad 1: Net-(D24-Pad2) -> r5
- SW24 pad 2: c3 -> Net-(D24-Pad2)
- SW25 pad 1: Net-(D25-Pad2) -> r0
- SW25 pad 2: c4 -> Net-(D25-Pad2)
- SW26 pad 1: Net-(D26-Pad2) -> r1
- SW26 pad 2: c4 -> Net-(D26-Pad2)
- SW27 pad 1: Net-(D27-Pad2) -> r2
- SW27 pad 2: c4 -> Net-(D27-Pad2)
- SW28 pad 1: Net-(D28-Pad2) -> r3
- SW28 pad 2: c4 -> Net-(D28-Pad2)
- SW29 pad 1: Net-(D29-Pad2) -> r4
- SW29 pad 2: c4 -> Net-(D29-Pad2)
- SW3 pad 1: Net-(D3-Pad2) -> r2
- SW3 pad 2: c0 -> Net-(D3-Pad2)
- SW30 pad 1: Net-(D30-Pad2) -> r5
- SW30 pad 2: c4 -> Net-(D30-Pad2)
- SW31 pad 1: Net-(D31-Pad2) -> r0
- SW31 pad 2: c5 -> Net-(D31-Pad2)
- SW32 pad 1: Net-(D32-Pad2) -> r1
- SW32 pad 2: c5 -> Net-(D32-Pad2)
- SW33 pad 1: Net-(D33-Pad2) -> r2
- SW33 pad 2: c5 -> Net-(D33-Pad2)
- SW34 pad 1: Net-(D34-Pad2) -> r3
- SW34 pad 2: c5 -> Net-(D34-Pad2)
- SW35 pad 1: Net-(D35-Pad2) -> r4
- SW35 pad 2: c5 -> Net-(D35-Pad2)
- SW36 pad 1: Net-(D36-Pad2) -> r5
- SW36 pad 2: c5 -> Net-(D36-Pad2)
- SW37 pad 1: Net-(D37-Pad2) -> r0
- SW37 pad 2: c6 -> Net-(D37-Pad2)
- SW38 pad 1: Net-(D38-Pad2) -> r1
- SW38 pad 2: c6 -> Net-(D38-Pad2)
- SW39 pad 1: Net-(D39-Pad2) -> r2
- SW39 pad 2: c6 -> Net-(D39-Pad2)
- SW4 pad 1: Net-(D4-Pad2) -> r3
- SW4 pad 2: c0 -> Net-(D4-Pad2)
- SW40 pad 1: Net-(D40-Pad2) -> r3
- SW40 pad 2: c6 -> Net-(D40-Pad2)
- SW41 pad 1: Net-(D41-Pad2) -> r4
- SW41 pad 2: c6 -> Net-(D41-Pad2)
- SW42 pad 1: Net-(D42-Pad2) -> r5
- SW42 pad 2: c6 -> Net-(D42-Pad2)
- SW43 pad 1: Net-(D43-Pad2) -> r0
- SW43 pad 2: c7 -> Net-(D43-Pad2)
- SW44 pad 1: Net-(D44-Pad2) -> r1
- SW44 pad 2: c7 -> Net-(D44-Pad2)
- SW45 pad 1: Net-(D45-Pad2) -> r2
- SW45 pad 2: c7 -> Net-(D45-Pad2)
- SW46 pad 1: Net-(D46-Pad2) -> r3
- SW46 pad 2: c7 -> Net-(D46-Pad2)
- SW47 pad 1: Net-(D47-Pad2) -> r4
- SW47 pad 2: c7 -> Net-(D47-Pad2)
- SW48 pad 1: Net-(D48-Pad2) -> r5
- SW48 pad 2: c7 -> Net-(D48-Pad2)
- SW49 pad 1: Net-(D49-Pad2) -> r0
- SW49 pad 2: c8 -> Net-(D49-Pad2)
- SW5 pad 1: Net-(D5-Pad2) -> r4
- SW5 pad 2: c0 -> Net-(D5-Pad2)
- SW50 pad 1: Net-(D50-Pad2) -> r1
- SW50 pad 2: c8 -> Net-(D50-Pad2)
- SW51 pad 1: Net-(D51-Pad2) -> r2
- SW51 pad 2: c8 -> Net-(D51-Pad2)
- SW52 pad 1: Net-(D52-Pad2) -> r3
- SW52 pad 2: c8 -> Net-(D52-Pad2)
- SW53 pad 1: Net-(D53-Pad2) -> r4
- SW53 pad 2: c8 -> Net-(D53-Pad2)
- SW54 pad 1: Net-(D54-Pad2) -> r5
- SW54 pad 2: c8 -> Net-(D54-Pad2)
- SW55 pad 1: Net-(D55-Pad2) -> r0
- SW55 pad 2: c9 -> Net-(D55-Pad2)
- SW56 pad 1: Net-(D56-Pad2) -> r1
- SW56 pad 2: c9 -> Net-(D56-Pad2)
- SW57 pad 1: Net-(D57-Pad2) -> r2
- SW57 pad 2: c9 -> Net-(D57-Pad2)
- SW58 pad 1: Net-(D58-Pad2) -> r3
- SW58 pad 2: c9 -> Net-(D58-Pad2)
- SW59 pad 1: Net-(D59-Pad2) -> r4
- SW59 pad 2: c9 -> Net-(D59-Pad2)
- SW6 pad 1: Net-(D6-Pad2) -> r5
- SW6 pad 2: c0 -> Net-(D6-Pad2)
- SW60 pad 1: Net-(D60-Pad2) -> r5
- SW60 pad 2: c9 -> Net-(D60-Pad2)
- SW61 pad 1: Net-(D61-Pad2) -> r0
- SW61 pad 2: c10 -> Net-(D61-Pad2)
- SW62 pad 1: Net-(D62-Pad2) -> r1
- SW62 pad 2: c10 -> Net-(D62-Pad2)
- SW63 pad 1: Net-(D63-Pad2) -> r2
- SW63 pad 2: c10 -> Net-(D63-Pad2)
- SW64 pad 1: Net-(D64-Pad2) -> r3
- SW64 pad 2: c10 -> Net-(D64-Pad2)
- SW65 pad 1: Net-(D65-Pad2) -> r4
- SW65 pad 2: c10 -> Net-(D65-Pad2)
- SW66 pad 1: Net-(D66-Pad2) -> r5
- SW66 pad 2: c10 -> Net-(D66-Pad2)
- SW67 pad 1: Net-(D67-Pad2) -> r0
- SW67 pad 2: c11 -> Net-(D67-Pad2)
- SW68 pad 1: Net-(D68-Pad2) -> r1
- SW68 pad 2: c11 -> Net-(D68-Pad2)
- SW69 pad 1: Net-(D69-Pad2) -> r2
- SW69 pad 2: c11 -> Net-(D69-Pad2)
- SW7 pad 1: Net-(D7-Pad2) -> r0
- SW7 pad 2: c1 -> Net-(D7-Pad2)
- SW70 pad 1: Net-(D70-Pad2) -> r3
- SW70 pad 2: c11 -> Net-(D70-Pad2)
- SW71 pad 1: Net-(D71-Pad2) -> r4
- SW71 pad 2: c11 -> Net-(D71-Pad2)
- SW72 pad 1: Net-(D72-Pad2) -> r5
- SW72 pad 2: c11 -> Net-(D72-Pad2)
- SW73 pad 1: Net-(D73-Pad2) -> r0
- SW73 pad 2: c12 -> Net-(D73-Pad2)
- SW74 pad 1: Net-(D74-Pad2) -> r1
- SW74 pad 2: c12 -> Net-(D74-Pad2)
- SW75 pad 1: Net-(D75-Pad2) -> r2
- SW75 pad 2: c12 -> Net-(D75-Pad2)
- SW76 pad 1: Net-(D76-Pad2) -> r3
- SW76 pad 2: c12 -> Net-(D76-Pad2)
- SW77 pad 1: Net-(D77-Pad2) -> r4
- SW77 pad 2: c12 -> Net-(D77-Pad2)
- SW78 pad 1: Net-(D78-Pad2) -> r5
- SW78 pad 2: c12 -> Net-(D78-Pad2)
- SW8 pad 1: Net-(D8-Pad2) -> r1
- SW8 pad 2: c1 -> Net-(D8-Pad2)
- SW9 pad 1: Net-(D9-Pad2) -> r2
- SW9 pad 2: c1 -> Net-(D9-Pad2)
Routing:
- net Net-(D68-Pad2): track 209.8 -> 4.74 mm, vias 1 -> 0
- net Net-(D69-Pad2): track 171.3 -> 4.74 mm, vias 1 -> 0
- net Net-(D62-Pad2): track 192.6 -> 37.7 mm, vias 1 -> 0
- net Net-(D63-Pad2): track 153.7 -> 4.74 mm, vias 1 -> 0
- net Net-(D70-Pad2): track 142.1 -> 4.74 mm, vias 1 -> 0
- net Net-(D56-Pad2): track 175.6 -> 41.5 mm, vias 1 -> 0
- net Net-(D64-Pad2): track 131.3 -> 4.74 mm, vias 1 -> 0
- net Net-(D42-Pad2): track 5.08 -> 130.6 mm
- net Net-(D6-Pad2): track 5.08 -> 129.1 mm
- net Net-(D12-Pad2): track 5.08 -> 127.2 mm
- net Net-(D36-Pad2): track 5.08 -> 126.1 mm
- net Net-(D18-Pad2): track 5.08 -> 125.3 mm
- net c6: track 229.4 -> 109.4 mm
- net Net-(D48-Pad2): track 5.08 -> 124.9 mm
- net Net-(D24-Pad2): track 5.08 -> 124.8 mm
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